Commit message: Added Simulator to the project

File: src/diy_robot_description/urdf/robot.urdf.xacro (robot description, xacro)
@@ -18,126 +18,237 @@
   All dimensions in metres, angles in radians.
 -->
-<robot name="diy_challenge_robot" xmlns:xacro="http://www.ros.org/wiki/xacro">
-  <!-- ═══════════════════════════════════════ MATERIALS ══ -->
-  <material name="dark_grey">
-    <color rgba="0.2 0.2 0.2 1.0"/>
+<robot xmlns:xacro="http://www.ros.org/wiki/xacro" name="juggernaut">
+  <!-- Define robot constants -->
+  <xacro:property name="base_off_ground" value="0.0714375"/> <!-- 2.8125 inches-->
+  <xacro:property name="base_width" value="0.346075"/> <!-- 13.625 inches-->
+  <xacro:property name="base_length" value="0.498475"/> <!-- 19.625 + 7.5 (pool noodle radius) inches-->
+  <xacro:property name="base_height" value="0.18415"/> <!-- 7.25 inches-->
+  <xacro:property name="pool_noodle_radius" value="0.047625"/> <!-- 1.875 inches-->
+  <xacro:property name="wheel_radius" value="0.09445625"/> <!-- 3.71875 inches-->
+  <xacro:property name="wheel_width" value="0.0508"/><!-- 2 inches-->
+  <xacro:property name="wheel_ygap" value="0.041275"/><!-- 1.625 inches-->
+  <xacro:property name="wheel_zoff" value="0.06985"/> <!-- 2.75 inches-->
+  <xacro:property name="drive_wheel_xoff" value="0.1254125"/><!-- 4.9375 inches-->
+  <xacro:property name="rear_wheel_xoff" value="0.1476375"/><!-- 5.8125 inches-->
+  <xacro:property name="camera_screw_zoff" value="-0.0385"/>
+  <xacro:property name="camera_screw_xoff" value="-0.007"/>
+  <!-- <xacro:property name="lidar_radius" value="0.038125"/>
+  <xacro:property name="lidar_length" value="0.076"/> --> <!-- old values defined as per the actual measurements -->
+  <xacro:property name="lidar_radius" value="0.0516"/>
+  <xacro:property name="lidar_length" value="0.0717"/>
+  <xacro:property name="imu_length" value="0.03"/>
+  <xacro:property name="imu_width" value="0.03"/>
+  <xacro:property name="imu_height" value="0.02"/>
+  <xacro:property name="hesai_centroid_y" value="-0.0298"/>
+  <xacro:property name="hesai_centroid_z" value="0.0124"/>
+  <xacro:arg name="use_nominal_extrinsics" default="true" />
+  <xacro:include filename="lidar.urdf.xacro" />
+  <xacro:include filename="imu.urdf.xacro" />
+  <xacro:lidar_3d_v1 parent="chassis" lidar_radius="${lidar_radius}" lidar_length="${lidar_length}">
+    <origin xyz="${base_length/2-lidar_radius} 0 ${base_height/2}" rpy="0 0 0" />
+   <!-- <origin xyz="0.569632 -0.03223 0.502056" rpy="0 0 0" /> -->
+  </xacro:lidar_3d_v1>
+  <xacro:imu_v1 parent="chassis" imu_length="${imu_length}" imu_width="${imu_width}" imu_height="${imu_height}">
+    <origin xyz="${base_length/2-lidar_radius} 0 0" rpy="0 0 0" />
+  </xacro:imu_v1>
+  <material name="transparent_blue">
+    <color rgba="0.0 0.0 1.0 0.25"/>
   </material>
   <material name="blue">
-    <color rgba="0.1 0.4 0.8 1.0"/>
+    <color rgba="0.0 0.0 1.0 1.0"/>
+  </material>
+  <material name="red">
+    <color rgba="1.0 0.0 0.0 1.0"/>
   </material>
   <material name="green">
-    <color rgba="0.1 0.8 0.2 1.0"/>
-  </material>
-  <material name="orange">
-    <color rgba="0.9 0.4 0.0 1.0"/>
-  </material>
-  <material name="white">
-    <color rgba="0.9 0.9 0.9 1.0"/>
-  </material>
-  <!-- ═══════════════════════════════════════ BASE LINK ══ -->
-  <link name="base_link">
-    <visual>
-      <geometry>
-        <box size="0.406 0.406 0.3"/>
-      </geometry>
-      <origin xyz="0 0 0.15" rpy="0 0 0"/>
-      <material name="dark_grey"/>
-    </visual>
-    <collision>
-      <geometry>
-        <box size="0.610 0.406 0.406"/>
-      </geometry>
-      <origin xyz="0 0 0.203" rpy="0 0 0"/>
-    </collision>
-    <inertial>
-      <mass value="8.0"/>
-      <inertia ixx="0.1" ixy="0.0" ixz="0.0"
-               iyy="0.1" iyz="0.0"
-               izz="0.1"/>
-    </inertial>
-  </link>
-  <!-- ═══════════════════════════════════════ LIDAR LINK ══
-       Hesai QT64 — mounted on top centre of chassis.
-       CALIB: Replace xyz and rpy with lidar_imu_calib extrinsic output.
-             extrinsic_T goes into xyz, extrinsic_R (Euler) into rpy. -->
-  <link name="lidar_link">
-    <visual>
-      <geometry>
-        <cylinder length="0.08" radius="0.06"/>
-      </geometry>
-      <material name="orange"/>
-    </visual>
-  </link>
-  <joint name="base_to_lidar" type="fixed">
-    <parent link="base_link"/>
-    <child link="lidar_link"/>
-    <!-- CALIB: Replace with lidar_imu_calib result for lidar→imu, then
-                compute imu→base_link to get this transform. -->
-    <origin xyz="0.0 0.0 0.38" rpy="0.0 0.0 0.0"/>
-  </joint>
-  <!-- ═══════════════════════════════════════ IMU LINK ══
-       Dedicated 6-DOF IMU (NOT the D435i built-in IMU).
-       CALIB: Replace with lidar_imu_calib extrinsic result.
-             This is the IMU→LiDAR transform inverse. -->
-  <link name="imu_link">
-    <visual>
-      <geometry>
-        <box size="0.03 0.03 0.015"/>
+    <color rgba="0.0 1.0 0.0 1.0"/>
+  </material>
+  <material name="Gray">
+    <color rgba="0.5 0.5 0.5 1.0"/>
+  </material>
+  <!-- Wheel xacro -->
+  <xacro:macro name="wheel" params="prefix x_reflect y_reflect wheel_xoff joint_type">
+    <link name="${prefix}_link">
+      <visual>
+        <origin xyz="0 0 0" rpy="${pi/2} 0 0"/>
+        <geometry>
+            <cylinder radius="${wheel_radius}" length="${wheel_width}"/>
+        </geometry>
+        <material name="red"/>
+      </visual>
+      <inertial>
+        <origin xyz="0 0 0" rpy="0 0 0"/>
+        <mass value="0.6"/>
+        <!-- solid cylinder around local Y (since we rotated the cylinder) -->
+        <inertia ixx="0.0012" ixy="0" ixz="0" iyy="0.0010" iyz="0" izz="0.0012"/>
+      </inertial>    <!-- ADD: collision matches visual -->
+      <collision>
+        <origin xyz="0 0 0" rpy="${pi/2} 0 0"/>
+        <geometry>
+          <cylinder radius="${wheel_radius}" length="${wheel_width}"/>
+        </geometry>
+        <!-- optional: stiffer contact so they don't sink -->
+        <surface>
+          <contact>
+            <ode>
+              <kp>1e6</kp>
+              <kd>1.0</kd>
+              <max_vel>0.1</max_vel>
+              <min_depth>0.001</min_depth>
+            </ode>
+          </contact>
+          <friction>
+            <ode>
+              <mu>1.0</mu>
+              <mu2>1.0</mu2>
+            </ode>
+          </friction>
+        </surface>
+      </collision>
+    </link>
+    <gazebo reference="${prefix}_link">
+        <material>Gazebo/Red</material>
+        <mu1>1.0</mu1>
+        <mu2>1.0</mu2>
+    </gazebo>
+    <joint name="${prefix}_joint" type="${joint_type}">
+      <parent link="chassis"/>
+      <child link="${prefix}_link"/>
+      <origin xyz="${x_reflect*wheel_xoff} ${y_reflect*(base_width/2+wheel_ygap)} ${-wheel_zoff}" rpy="0 0 0"/>
+      <axis xyz="0 1 0"/>
+    </joint>
+  </xacro:macro>
+  <link name="base_footprint"/>
+  <joint name="base_footprint_to_chassis" type="fixed">
+    <parent link="base_footprint"/>
+    <child link="chassis"/>
+    <origin xyz="0 0 ${(wheel_radius+wheel_zoff)}" rpy="0 0 0"/>
+  </joint>
+  <link name="chassis">
+    <inertial>
+      <origin xyz="0 0 0" rpy="0 0 0"/> <!-- change based on TF -->
+      <mass value="10.0"/>
+      <inertia ixx="0.128066" ixy="0.0" ixz="0.0" iyy="0.235324" iyz="0.0" izz="0.306871"/>
+    </inertial>
+    <visual>
+      <origin xyz="0 0 0" rpy="0 0 0"/>
+      <geometry>
+        <box size="${base_length} ${base_width} ${base_height}"/>
+      </geometry>
+      <material name="transparent_blue"/>
+    </visual>
+    <collision>
+      <origin xyz="0 0 0" rpy="0 0 0"/> <!-- change based on TF -->
+      <geometry>
+        <box size="${base_length} ${base_width} ${base_height}"/>
+      </geometry>
+    </collision>
+  </link>
+  <xacro:wheel prefix="drivewhl_l" x_reflect="1" y_reflect="1" wheel_xoff="${drive_wheel_xoff}" joint_type="continuous"/>
+  <xacro:wheel prefix="drivewhl_r" x_reflect="1" y_reflect="-1" wheel_xoff="${drive_wheel_xoff}" joint_type="continuous"/>
+  <xacro:wheel prefix="rearwhl_l" x_reflect="-1" y_reflect="1" wheel_xoff="${rear_wheel_xoff}" joint_type="continuous"/>
+  <xacro:wheel prefix="rearwhl_r" x_reflect="-1" y_reflect="-1" wheel_xoff="${rear_wheel_xoff}" joint_type="continuous"/>
+<!--
+  <link name="wheel_1">
+    <inertial>
+      <origin xyz="0 0 0" rpy="0 0 0"/>
+      <mass value="2.0"/>
+      <inertia ixx="0.145833" ixy="0.0" ixz="0.0" iyy="0.145833" iyz="0.0" izz="0.125"/>
+    </inertial>
+    <visual>
+      <origin xyz="0 0 0" rpy="0 0 0"/>
+      <geometry>
+        <cylinder radius="0.3" length="0.25"/>
+      </geometry>
+      <material name="red"/>
+    </visual>
+    <collision>
+      <origin xyz="0 0 0" rpy="0 0 0"/>
+      <geometry>
+        <cylinder radius="0.3" length="0.25"/>
+      </geometry>
+    </collision>
+  </link>
+  <joint name="chassis_wheel_1_revolute" type="continuous">
+    <parent link="chassis"/>
+    <child link="wheel_1"/>
+    <origin xyz="0.554283 0.625029 -0.025" rpy="1.57079632679 0 0"/>
+    <axis xyz="0 0 1"/>
+    <dynamics damping="0.0" friction="0.0"/>
+  </joint>
+  <link name="wheel_2">
+    <inertial>
+      <origin xyz="0 0 0" rpy="0 0 0"/>
+      <mass value="2.0"/>
+      <inertia ixx="0.145833" ixy="0.0" ixz="0.0" iyy="0.145833" iyz="0.0" izz="0.125"/>
+    </inertial>
+    <visual>
+      <origin xyz="0 0 0" rpy="0 0 0"/>
+      <geometry>
+        <cylinder radius="0.3" length="0.25"/>
+      </geometry>
+      <material name="red"/>
+    </visual>
+    <collision>
+      <origin xyz="0 0 0" rpy="0 0 0"/>
+      <geometry>
+        <cylinder radius="0.3" length="0.25"/>
+      </geometry>
+    </collision>
+  </link>
+  <joint name="chassis_wheel_2_revolute" type="continuous">
+    <parent link="chassis"/>
+    <child link="wheel_2"/>
+    <origin xyz="0.554282 -0.625029 -0.025" rpy="1.57079632679 0 0"/>
+    <axis xyz="0 0 1"/>
+    <dynamics damping="0.0" friction="0.0"/>
+  </joint>
+  <link name="caster">
+    <inertial>
+      <origin xyz="0 0 0" rpy="0 0 0"/>
+      <mass value="1.0"/>
+      <inertia ixx="0.1" ixy="0.0" ixz="0.0" iyy="0.1" iyz="0.0" izz="0.1"/>
+    </inertial>
+    <visual>
+      <origin xyz="0 0 0" rpy="0 0 0"/>
+      <geometry>
+        <sphere radius="0.2"/>
       </geometry>
       <material name="green"/>
     </visual>
-  </link>
-  <joint name="base_to_imu" type="fixed">
-    <parent link="base_link"/>
-    <child link="imu_link"/>
-    <!-- CALIB: Replace with measured/calibrated IMU mount position. -->
-    <origin xyz="0.0 0.0 0.25" rpy="0.0 0.0 0.0"/>
-  </joint>
-  <!-- ═══════════════════════════════════════ CAMERA LINK ══
-       RealSense D435i — mounted front of chassis, facing forward.
-       CALIB: Replace with cam_lidar_calib extrinsic result.
-             camera_link is the standard RealSense optical frame origin. -->
-  <link name="camera_link">
-    <visual>
-      <geometry>
-        <box size="0.09 0.025 0.025"/>
-      </geometry>
-      <material name="blue"/>
-    </visual>
-  </link>
-  <joint name="base_to_camera" type="fixed">
-    <parent link="base_link"/>
-    <child link="camera_link"/>
-    <!-- CALIB: Replace xyz with measured mount position.
-                rpy: camera faces forward (+x of base_link), need
-                RealSense→ROS optical convention if using stereo topics. -->
-    <origin xyz="0.20 0.0 0.20" rpy="0.0 0.0 0.0"/>
-  </joint>
-  <!-- Camera optical frame (required by apriltag_ros and realsense2_ros) -->
-  <link name="camera_optical_link"/>
-  <joint name="camera_to_optical" type="fixed">
-    <parent link="camera_link"/>
-    <child link="camera_optical_link"/>
-    <!-- ROS optical convention: x right, y down, z into scene -->
-    <origin xyz="0 0 0" rpy="-1.5707963 0 -1.5707963"/>
-  </joint>
-  <!-- ═══════════════════════════════════════ GPS LINK ══
-       RTK GNSS antenna phase centre.
-       CALIB: Physically measure the 3D offset from antenna phase centre
-              to base_link origin (geometric centre at floor level).
-              An uncompensated 10 cm lever arm causes systematic heading error. -->
-  <link name="gps_link">
-    <visual>
-      <geometry>
-        <cylinder length="0.02" radius="0.04"/>
-      </geometry>
-      <material name="white"/>
-    </visual>
-  </link>
-  <joint name="base_to_gps" type="fixed">
-    <parent link="base_link"/>
-    <child link="gps_link"/>
-    <!-- CALIB: Replace with physically measured antenna phase centre position. -->
-    <origin xyz="0.0 0.0 0.42" rpy="0.0 0.0 0.0"/>
-  </joint>
+    <collision>
+      <origin xyz="0 0 0" rpy="0 0 0"/>
+      <geometry>
+        <sphere radius="0.2"/>
+      </geometry>
+    </collision>
+  </link>
+  <joint name="chassis_caster_ball" type="fixed">
+    <parent link="chassis"/>
+    <child link="caster"/>
+    <origin xyz="-0.957138 0.0 -0.125" rpy="0 0 0"/>
+  </joint>
+  <gazebo reference="chassis">
+    <material>Gazebo/Blue</material>
+    <mu1>1.0</mu1>
+    <mu2>1.0</mu2>
+  </gazebo>
+  <gazebo reference="wheel_1">
+    <material>Gazebo/Red</material>
+    <mu1>1.0</mu1>
+    <mu2>1.0</mu2>
+  </gazebo>
+  <gazebo reference="wheel_2">
+    <material>Gazebo/Red</material>
+    <mu1>1.0</mu1>
+    <mu2>1.0</mu2>
+  </gazebo>
+  <gazebo reference="caster">
+    <material>Gazebo/Green</material>
+    <mu1>0.0</mu1>
+    <mu2>0.0</mu2>
+    <slip1>1.0</slip1>
+    <slip2>1.0</slip2>
+  </gazebo>
+-->
 </robot>
