Commit message: Udated Robot Xacro

File: src/diy_robot_description/urdf/robot.urdf.xacro (robot description, xacro)
@@ -10,9 +10,10 @@
     map
      └── odom            (published by navsat_transform / EKF2)
-          └── base_link  (published by EKF1 via /odometry/filtered)
-               ├── lidar_link   <- fixed, from lidar_imu_calib
-               ├── imu_link     <- fixed, from lidar_imu_calib
-               ├── camera_link  <- fixed, from cam_lidar_calib
-               └── gps_link     <- fixed, measured lever arm
+          └── base_footprint  (published by EKF2 via /odometry/filtered)
+               └──base_link  (published by URDF via robot_state_publisher)
+                    ├── lidar_link   <- fixed, from lidar_imu_calib
+                    ├── imu_link     <- fixed, from lidar_imu_calib
+                    ├── camera_link  <- fixed, from cam_lidar_calib
+                    └── gps_link     <- fixed, measured lever arm
   Robot body: 406 mm L × 406 mm W × 406 mm H (16" × 16" × 16")
   All dimensions in metres, angles in radians.
@@ -34,4 +35,24 @@
   <xacro:property name="camera_screw_zoff" value="-0.0385"/>
   <xacro:property name="camera_screw_xoff" value="-0.007"/>
+  <!-- New Values-->
+  <xacro:property name="body_mass" value="10.0"/> <!-- in Kg-->
+  <xacro:property name="base_off_ground" value="0.0523875"/> <!-- 2.0625 inches-->
+  <xacro:property name="base_width" value="0.2159"/> <!-- 8.5 inches (chassis only; total width incl. wheels = 16 in / 0.4064 m)-->
+  <xacro:property name="base_length" value="0.419735"/> <!-- 16.525 inches-->
+  <xacro:property name="base_height" value="0.1524"/> <!-- 6 inches-->
+  <xacro:property name="pool_noodle_radius" value="0.047625"/> <!-- 1.875 inches-->
+  <xacro:property name="wheel_radius" value="0.0762"/> <!-- 3 inches-->
+  <xacro:property name="wheel_width" value="0.0254"/><!-- 1 inches-->
+  <xacro:property name="wheel_ygap" value="0.016256"/><!-- 0.64 inches-->
+  <xacro:property name="wheel_zoff" value="0.0"/> <!-- 0 inches-->
+  <xacro:property name="drive_wheel_xoff" value="0.0"/><!-- 0 inches-->
+  <xacro:property name="rear_wheel_xoff" value="0.2794"/><!-- 11 inches-->
+  <xacro:property name="castor_wheel_radius" value="0.01"/> <!-- 3.71875 inches-->
+  <xacro:property name="sensor_xoff_from_AR" value="0.072644"/> <!-- 2.86 inches-->
+  <xacro:property name="Lidar_base_height_from_AR" value="0.1285875"/> <!-- 5.0625 inches-->
+  <xacro:property name="imu_height_from_AR" value="0.0333375"/> <!-- 1.3125 inches-->
+  <xacro:property name="AR_from_front" value="0.0964565"/> <!-- 3.7975 inches-->
+  <xacro:property name="camera_screw_zoff" value="-0.0385"/>
+  <xacro:property name="camera_screw_xoff" value="-0.007"/>
   <!-- <xacro:property name="lidar_radius" value="0.038125"/>
   <xacro:property name="lidar_length" value="0.076"/> --> <!-- old values defined as per the actual measurements -->
@@ -46,10 +67,10 @@
   <xacro:include filename="lidar.urdf.xacro" />
   <xacro:include filename="imu.urdf.xacro" />
-  <xacro:lidar_3d_v1 parent="chassis" lidar_radius="${lidar_radius}" lidar_length="${lidar_length}">
-    <origin xyz="${base_length/2-lidar_radius} 0 ${base_height/2}" rpy="0 0 0" />
+  <xacro:lidar_3d_v1 parent="base_link" lidar_radius="${lidar_radius}" lidar_length="${lidar_length}">
+    <origin xyz="${sensor_xoff_from_AR} 0 ${Lidar_base_height_from_AR}" rpy="0 0 0" />
    <!-- <origin xyz="0.569632 -0.03223 0.502056" rpy="0 0 0" /> -->
   </xacro:lidar_3d_v1>
-  <xacro:imu_v1 parent="chassis" imu_length="${imu_length}" imu_width="${imu_width}" imu_height="${imu_height}">
-    <origin xyz="${base_length/2-lidar_radius} 0 0" rpy="0 0 0" />
+  <xacro:imu_v1 parent="base_link" imu_length="${imu_length}" imu_width="${imu_width}" imu_height="${imu_height}">
+    <origin xyz="${sensor_xoff_from_AR} 0 ${imu_height_from_AR}" rpy="0 0 0" />
   </xacro:imu_v1>
   <material name="transparent_blue">
@@ -116,5 +137,5 @@
     </gazebo>
     <joint name="${prefix}_joint" type="${joint_type}">
-      <parent link="chassis"/>
+      <parent link="base_link"/>
       <child link="${prefix}_link"/>
       <origin xyz="${x_reflect*wheel_xoff} ${y_reflect*(base_width/2+wheel_ygap)} ${-wheel_zoff}" rpy="0 0 0"/>
@@ -124,17 +145,25 @@
   </xacro:macro>
   <link name="base_footprint"/>
-  <joint name="base_footprint_to_chassis" type="fixed">
+  <joint name="base_footprint_to_base_link" type="fixed">
     <parent link="base_footprint"/>
+    <child link="base_link"/>
+    <origin xyz="0 0 ${wheel_radius}" rpy="0 0 0"/>
+  </joint>
+  <link name="base_link"/>
+  <joint name="base_link_to_chassis" type="fixed">
+    <parent link="base_link"/>
     <child link="chassis"/>
-    <origin xyz="0 0 ${(wheel_radius+wheel_zoff)}" rpy="0 0 0"/>
+    <origin xyz="${AR_from_front-base_length/2} 0 ${base_height/2+base_off_ground-wheel_radius}" rpy="0 0 0"/>
   </joint>
   <link name="chassis">
     <inertial>
-      <origin xyz="0 0 0" rpy="0 0 0"/> <!-- change based on TF -->
-      <mass value="10.0"/>
-      <inertia ixx="0.128066" ixy="0.0" ixz="0.0" iyy="0.235324" iyz="0.0" izz="0.306871"/>
-    </inertial>
-    <visual>
-      <origin xyz="0 0 0" rpy="0 0 0"/>
+      <origin xyz="${AR_from_front-base_length/2} 0 ${base_height/2+base_off_ground-wheel_radius}" rpy="0 0 0"/> <!-- change based on TF -->
+      <mass value="${body_mass}"/>
+      <inertia ixx="0.5 * body_mass * (base_width * base_width + base_height * base_height)" ixy="0.0" ixz="0.0"
+               iyy="0.5 * body_mass * (base_length * base_length + base_height * base_height)" iyz="0.0"
+               izz="0.5 * body_mass * (base_length * base_length + base_width * base_width)"/>
+    </inertial>
+    <visual>
+      <origin xyz="${AR_from_front-base_length/2} 0 ${base_height/2+base_off_ground-wheel_radius}" rpy="0 0 0"/>
       <geometry>
         <box size="${base_length} ${base_width} ${base_height}"/>
@@ -143,5 +172,5 @@
     </visual>
     <collision>
-      <origin xyz="0 0 0" rpy="0 0 0"/> <!-- change based on TF -->
+      <origin xyz="${AR_from_front-base_length/2} 0 ${base_height/2+base_off_ground-wheel_radius}" rpy="0 0 0"/> <!-- change based on TF -->
       <geometry>
         <box size="${base_length} ${base_width} ${base_height}"/>

Commit message: Caster wheel update

File: src/diy_robot_description/urdf/robot.urdf.xacro (robot description, xacro)
@@ -199,5 +199,5 @@
   </link>
   <joint name="chassis_caster_ball" type="continuous">
-    <parent link="chassis"/>
+    <parent link="base_link"/>
     <child link="caster"/>
     <origin xyz="${-1*rear_wheel_xoff} 0.0 ${-1*wheel_zoff}" rpy="0 0 0"/>

Commit message: updated xacro

File: src/diy_robot_description/urdf/robot.urdf.xacro (robot description, xacro)
@@ -21,36 +21,22 @@
 <robot xmlns:xacro="http://www.ros.org/wiki/xacro" name="juggernaut">
   <!-- Define robot constants -->
-  <xacro:property name="base_off_ground" value="0.0714375"/> <!-- 2.8125 inches-->
-  <xacro:property name="base_width" value="0.27305"/> <!-- 10.75 inches (chassis only; total width incl. wheels = 16 in / 0.4064 m)-->
-  <xacro:property name="base_length" value="0.498475"/> <!-- 19.625 + 7.5 (pool noodle radius) inches-->
-  <xacro:property name="base_height" value="0.18415"/> <!-- 7.25 inches-->
-  <xacro:property name="pool_noodle_radius" value="0.047625"/> <!-- 1.875 inches-->
-  <xacro:property name="wheel_radius" value="0.09445625"/> <!-- 3.71875 inches-->
-  <xacro:property name="wheel_width" value="0.0508"/><!-- 2 inches-->
-  <xacro:property name="wheel_ygap" value="0.041275"/><!-- 1.625 inches-->
-  <xacro:property name="wheel_zoff" value="0.06985"/> <!-- 2.75 inches-->
-  <xacro:property name="drive_wheel_xoff" value="0.1254125"/><!-- 4.9375 inches-->
-  <xacro:property name="rear_wheel_xoff" value="0.1476375"/><!-- 5.8125 inches-->
-  <xacro:property name="castor_wheel_radius" value="0.01"/> <!-- 3.71875 inches-->
-  <xacro:property name="camera_screw_zoff" value="-0.0385"/>
-  <xacro:property name="camera_screw_xoff" value="-0.007"/>
   <!-- New Values-->
-  <xacro:property name="body_mass" value="10.0"/> <!-- in Kg-->
-  <xacro:property name="base_off_ground" value="0.0523875"/> <!-- 2.0625 inches-->
-  <xacro:property name="base_width" value="0.2159"/> <!-- 8.5 inches (chassis only; total width incl. wheels = 16 in / 0.4064 m)-->
-  <xacro:property name="base_length" value="0.419735"/> <!-- 16.525 inches-->
-  <xacro:property name="base_height" value="0.1524"/> <!-- 6 inches-->
+  <xacro:property name="body_mass" value="9.470"/> <!-- in Kg-->
+  <xacro:property name="base_off_ground" value="0.0508"/> <!-- 2.0 inches / -->
+  <xacro:property name="base_width" value="0.2145665"/> <!-- 8.4475 inches (chassis only; total width incl. wheels = 16 in / 0.4064 m)-->
+  <xacro:property name="base_length" value="0.4318"/> <!-- 17 inches-->
+  <xacro:property name="base_height" value="0.174625"/> <!-- 6.875 inches-->
   <xacro:property name="pool_noodle_radius" value="0.047625"/> <!-- 1.875 inches-->
   <xacro:property name="wheel_radius" value="0.0762"/> <!-- 3 inches-->
   <xacro:property name="wheel_width" value="0.0254"/><!-- 1 inches-->
-  <xacro:property name="wheel_ygap" value="0.016256"/><!-- 0.64 inches-->
-  <xacro:property name="wheel_zoff" value="0.0"/> <!-- 0 inches-->
+  <xacro:property name="wheel_ygap" value="0.0174625"/><!-- 0.6875 inches-->
+  <xacro:property name="wheel_zoff" value="-0.0619125"/> <!-- -2.4375 inches-->
   <xacro:property name="drive_wheel_xoff" value="0.0"/><!-- 0 inches-->
   <xacro:property name="rear_wheel_xoff" value="0.2794"/><!-- 11 inches-->
-  <xacro:property name="castor_wheel_radius" value="0.01"/> <!-- 3.71875 inches-->
-  <xacro:property name="sensor_xoff_from_AR" value="0.072644"/> <!-- 2.86 inches-->
-  <xacro:property name="Lidar_base_height_from_AR" value="0.1285875"/> <!-- 5.0625 inches-->
+  <xacro:property name="castor_wheel_radius" value="0.0762"/> <!-- 3.0inches-->
+  <xacro:property name="sensor_xoff_from_AR" value="0.0568325"/> <!-- 2.2375 inches-->
+  <xacro:property name="Lidar_base_height_from_AR" value="0.149225"/> <!-- 5.875 inches-->
   <xacro:property name="imu_height_from_AR" value="0.0333375"/> <!-- 1.3125 inches-->
-  <xacro:property name="AR_from_front" value="0.0964565"/> <!-- 3.7975 inches-->
+  <xacro:property name="AR_from_front" value="0.0771525"/> <!-- 3.0375 inches-->
   <xacro:property name="camera_screw_zoff" value="-0.0385"/>
   <xacro:property name="camera_screw_xoff" value="-0.007"/>
