Commit message: WIP fast lio still drifting a lot

File: src/diy_robot_description/urdf/lidar.urdf.xacro (robot description, xacro)
@@ -42,6 +42,6 @@
               <samples>640</samples>
               <resolution>1</resolution>
-              <min_angle>-1.5708</min_angle>
-              <max_angle>1.5708</max_angle>
+              <min_angle>-3.141592653589793</min_angle>
+              <max_angle>3.141592653589793</max_angle>
             </horizontal>
             <vertical>

File: src/diy_robot_description/urdf/robot.urdf.xacro (robot description, xacro)
@@ -28,5 +28,5 @@
   <xacro:property name="wheel_width" value="0.0508"/><!-- 2 inches-->
   <xacro:property name="wheel_ygap" value="0.041275"/><!-- 1.625 inches-->
-  <xacro:property name="wheel_zoff" value="0.06985"/> <!-- 2.75 inches-->
+  <xacro:property name="wheel_zoff" value="${base_off_ground + base_height/2 - wheel_radius}"/> <!-- derived from chassis ground clearance -->
   <xacro:property name="drive_wheel_xoff" value="0.1254125"/><!-- 4.9375 inches-->
   <xacro:property name="rear_wheel_xoff" value="0.1476375"/><!-- 5.8125 inches-->
@@ -46,9 +46,9 @@
   <xacro:include filename="lidar.urdf.xacro" />
   <xacro:include filename="imu.urdf.xacro" />
-  <xacro:lidar_3d_v1 parent="chassis" lidar_radius="${lidar_radius}" lidar_length="${lidar_length}">
+  <xacro:lidar_3d_v1 parent="base_link" lidar_radius="${lidar_radius}" lidar_length="${lidar_length}">
     <origin xyz="${base_length/2-lidar_radius} 0 ${base_height/2}" rpy="0 0 0" />
    <!-- <origin xyz="0.569632 -0.03223 0.502056" rpy="0 0 0" /> -->
   </xacro:lidar_3d_v1>
-  <xacro:imu_v1 parent="chassis" imu_length="${imu_length}" imu_width="${imu_width}" imu_height="${imu_height}">
+  <xacro:imu_v1 parent="base_link" imu_length="${imu_length}" imu_width="${imu_width}" imu_height="${imu_height}">
     <origin xyz="${base_length/2-lidar_radius} 0 0" rpy="0 0 0" />
   </xacro:imu_v1>
@@ -114,5 +114,5 @@
     </gazebo>
     <joint name="${prefix}_joint" type="${joint_type}">
-      <parent link="chassis"/>
+      <parent link="base_link"/>
       <child link="${prefix}_link"/>
       <origin xyz="${x_reflect*wheel_xoff} ${y_reflect*(base_width/2+wheel_ygap)} ${-wheel_zoff}" rpy="0 0 0"/>
@@ -120,11 +120,5 @@
     </joint>
   </xacro:macro>
-  <link name="base_footprint"/>
-  <joint name="base_footprint_to_chassis" type="fixed">
-    <parent link="base_footprint"/>
-    <child link="chassis"/>
-    <origin xyz="0 0 ${(wheel_radius+wheel_zoff)}" rpy="0 0 0"/>
-  </joint>
-  <link name="chassis">
+  <link name="base_link">
     <inertial>
       <origin xyz="0 0 0" rpy="0 0 0"/> <!-- change based on TF -->
@@ -166,6 +160,6 @@
     </collision>
   </link>
-  <joint name="chassis_caster_ball" type="continuous">
-    <parent link="chassis"/>
+  <joint name="base_link_caster_ball" type="continuous">
+    <parent link="base_link"/>
     <child link="caster"/>
     <origin xyz="${-1*rear_wheel_xoff} 0.0 ${-1*wheel_zoff}" rpy="0 0 0"/>
@@ -177,5 +171,5 @@
   -->
   <gazebo>
-    <plugin filename="gz-sim-diff-drive-system" name="gz::sim::systems::DiffDrive">
+    <plugin filename="libignition-gazebo-diff-drive-system.so" name="ignition::gazebo::systems::DiffDrive">
         <left_joint>drivewhl_l_joint</left_joint>
         <right_joint>drivewhl_r_joint</right_joint>
@@ -187,5 +181,5 @@
   </gazebo>
   <gazebo>
-    <plugin filename="gz-sim-joint-state-publisher-system" name="gz::sim::systems::JointStatePublisher">
+    <plugin filename="libignition-gazebo-joint-state-publisher-system.so" name="ignition::gazebo::systems::JointStatePublisher">
         <topic>joint_states</topic> <joint_name>drivewhl_l_joint</joint_name>
         <joint_name>drivewhl_r_joint</joint_name>
@@ -194,6 +188,6 @@
    <!-- INSERT GROUND TRUTH POSE PUBLISHER HERE -->
   <gazebo>
-    <plugin filename="libignition-gazebo-pose-publisher-system.so"
-          name="ignition::gazebo::systems::PosePublisher">
+      <plugin filename="libignition-gazebo-pose-publisher-system.so"
+        name="ignition::gazebo::systems::PosePublisher">
       <publish_link_pose>false</publish_link_pose>
       <publish_visual_pose>false</publish_visual_pose>

Commit message: feat: switch to RPP-ready nav pipeline with in-place rotation circuit runner
- nav2_params.yaml: switch planner SmacHybrid→NavfnPlanner, tune MPPI critics
  (PathAlignCritic, ObstaclesCritic, GoalAngleCritic), reduce global inflation
  0.30→0.15m for 1.05m corridors, yaw_goal_tolerance relaxed for circuit_runner
- circuit_runner_node.py: rewrite to use NavigateToPose per waypoint with
  rotate_in_place mode — pure cmd_vel angular spin at corners, bypassing MPPI
- sim_simple_loop_waypoints.yaml: simplified to 4 corner waypoints with
  rotate_in_place:true; turns placed 2m before walls to avoid inflation zone
- behavior_trees/: add custom Spin-free BT XMLs to fix bt_navigator crash
- sim_nav.launch.py: new launch file for sim-only Nav2 bringup
- simple_loop.sdf: new rectangular test world (1.05m corridors, 13x13m loop)
- sim_competition.launch.py, sim_telemetry.py: competition sim infra
- competition_arena.sdf: updated obstacle course world geometry
- keepout_mask: add global costmap keepout filter map
- record_trajectory.py: diagnostic script with stuck zone detection
- robot.urdf.xacro, lidar.urdf.xacro: minor URDF fixes
- docs/: add 2026 Course Layouts PDF; remove stale arch diagrams

File: src/diy_robot_description/urdf/lidar.urdf.xacro (robot description, xacro)
@@ -34,5 +34,5 @@
         <always_on>true</always_on>
         <update_rate>10</update_rate>
-        <visualize>true</visualize>
+        <visualize>false</visualize>
         <topic>lidar</topic>
         <ignition_frame_id>lidar_link</ignition_frame_id>

File: src/diy_robot_description/urdf/robot.urdf.xacro (robot description, xacro)
@@ -21,5 +21,5 @@
   <!-- Define robot constants -->
   <xacro:property name="base_off_ground" value="0.0714375"/> <!-- 2.8125 inches-->
-  <xacro:property name="base_width" value="0.346075"/> <!-- 13.625 inches-->
+  <xacro:property name="base_width" value="0.27305"/> <!-- 10.75 inches (chassis only; total width incl. wheels = 16 in / 0.4064 m)-->
   <xacro:property name="base_length" value="0.498475"/> <!-- 19.625 + 7.5 (pool noodle radius) inches-->
   <xacro:property name="base_height" value="0.18415"/> <!-- 7.25 inches-->
@@ -110,6 +110,8 @@
     <gazebo reference="${prefix}_link">
         <material>Gazebo/Red</material>
-        <mu1>1.0</mu1>
-        <mu2>1.0</mu2>
+        <mu1>1.5</mu1>
+        <mu2>1.5</mu2>
+        <kp>1e6</kp>
+        <kd>1.0</kd>
     </gazebo>
     <joint name="${prefix}_joint" type="${joint_type}">
@@ -118,4 +120,5 @@
       <origin xyz="${x_reflect*wheel_xoff} ${y_reflect*(base_width/2+wheel_ygap)} ${-wheel_zoff}" rpy="0 0 0"/>
       <axis xyz="0 1 0"/>
+      <limit effort="20.0" velocity="10.0"/>
     </joint>
   </xacro:macro>
@@ -183,5 +186,24 @@
         <wheel_radius>${wheel_radius}</wheel_radius>     <!-- Adjust to your wheel radius (meters) -->
         <topic>cmd_vel</topic>
+        <odom_topic>odom_wheel</odom_topic>   <!-- wheel encoder odom — drifts on ramp/slip -->
+        <!-- Publish odom→base_footprint TF — must match Nav2 robot_base_frame.
+             Ignition namespaces these as diy_robot/odom→diy_robot/base_footprint.
+             SIM only: on real robot EKF1/EKF2 publish this transform instead. -->
+        <odom_frame>odom</odom_frame>
+        <robot_base_frame>base_footprint</robot_base_frame>
+        <tf_topic>/tf</tf_topic>
         <robot_param_node>/robot_state_publisher</robot_param_node>
+    </plugin>
+  </gazebo>
+  <!-- SIM ONLY: Ground-truth odometry from Gazebo physics engine.
+       Publishes perfect pose to /odom — no wheel slip drift.
+       On real robot: EKF2 fuses wheel + IMU + NDT into /odometry/filtered instead. -->
+  <gazebo>
+    <plugin filename="gz-sim-odometry-publisher-system" name="gz::sim::systems::OdometryPublisher">
+        <odom_frame>odom</odom_frame>
+        <robot_base_frame>base_footprint</robot_base_frame>
+        <odom_topic>/odom</odom_topic>
+        <tf_topic>/tf</tf_topic>
+        <odom_publish_frequency>50</odom_publish_frequency>
     </plugin>
   </gazebo>
