Commit message: Update pure pursuit controller and navigation launch

File: src/diy_robot_description/urdf/original.urdf.xacro (robot description, xacro)
@@ -31,6 +31,5 @@
   <xacro:property name="drive_wheel_xoff" value="0.1254125"/><!-- 4.9375 inches-->
   <xacro:property name="rear_wheel_xoff" value="0.1476375"/><!-- 5.8125 inches-->
-  <xacro:property name="castor_wheel_radius" value="0.1016"/> <!-- 4-inch radius / 8-inch diameter -->
-  <xacro:property name="castor_wheel_width" value="0.0574"/> <!-- 2.26-inch STL depth -->
+  <xacro:property name="castor_wheel_radius" value="0.01"/> <!-- 3.71875 inches-->
   <xacro:property name="camera_screw_zoff" value="-0.0385"/>
   <xacro:property name="camera_screw_xoff" value="-0.007"/>
@@ -124,66 +123,5 @@
     </joint>
   </xacro:macro>
-  <!-- Rear omni wheel xacro: fixed axle, passive wheel rotation.
-       The wheel does NOT swivel. Omni behavior is approximated with
-       high friction in the rolling direction (X) and low friction
-       laterally along the axle direction (Y). -->
-  <xacro:macro name="rear_caster" params="prefix x_reflect y_reflect wheel_xoff joint_type">
-    <link name="${prefix}_link">
-      <visual>
-        <origin xyz="-0.093339143 0.185046036 -0.156049187"
-                rpy="${pi/2} 0 0"/>
-        <geometry>
-          <mesh filename="package://diy_robot_description/urdf/meshes/caster_wheel.stl"
-                scale="0.0254 0.0254 0.0254"/>
-        </geometry>
-        <material name="green"/>
-      </visual>
-      <inertial>
-        <origin xyz="0 0 0" rpy="0 0 0"/>
-        <mass value="0.6"/>
-        <inertia ixx="0.0012" ixy="0" ixz="0"
-                 iyy="0.0010" iyz="0" izz="0.0012"/>
-      </inertial>
-      <!-- Simple cylindrical collision for the omni wheel.
-           The roller effect is represented by anisotropic friction below. -->
-      <collision>
-        <origin xyz="0 0 0" rpy="${pi/2} 0 0"/>
-        <geometry>
-          <cylinder radius="${castor_wheel_radius}" length="${castor_wheel_width}"/>
-        </geometry>
-      </collision>
-    </link>
-    <!-- Fixed wheel orientation: only the wheel spins about its axle (Y). -->
-    <joint name="${prefix}_joint" type="${joint_type}">
-      <parent link="chassis"/>
-      <child link="${prefix}_link"/>
-      <origin xyz="${x_reflect*wheel_xoff} ${y_reflect*(base_width/2+wheel_ygap)} ${-wheel_zoff}" rpy="0 0 0"/>
-      <axis xyz="0 1 0"/>
-      <dynamics damping="0.02" friction="0.0"/>
-      <limit effort="20.0" velocity="20.0"/>
-    </joint>
-    <!-- Omni-wheel approximation:
-         fdir1 = chassis/wheel X direction
-         mu1   = normal rolling-direction traction
-         mu2   = very low lateral resistance along Y, emulating free rollers -->
-    <gazebo reference="${prefix}_link">
-      <material>Gazebo/Green</material>
-      <mu1>1.0</mu1>
-      <mu2>0.02</mu2>
-      <fdir1>1 0 0</fdir1>
-      <kp>1e6</kp>
-      <kd>1.0</kd>
-      <slip1>0.0</slip1>
-      <slip2>1.0</slip2>
-    </gazebo>
-  </xacro:macro>
-  <link name="base_footprint">
-    <inertial>
-      <mass value="0.001"/>
-      <inertia ixx="1e-06" ixy="0.0" ixz="0.0"
-               iyy="1e-06" iyz="0.0"
-               izz="1e-06"/>
-    </inertial>
-  </link>
+  <link name="base_footprint"/>
   <joint name="base_footprint_to_chassis" type="fixed">
     <parent link="base_footprint"/>
@@ -211,8 +149,34 @@
     </collision>
   </link>
+  <link name="caster">
+    <inertial>
+      <origin xyz="0 0 0" rpy="0 0 0"/>
+      <mass value="1.0"/>
+      <inertia ixx="0.1" ixy="0.0" ixz="0.0" iyy="0.1" iyz="0.0" izz="0.1"/>
+    </inertial>
+    <visual>
+      <origin xyz="0 0 0" rpy="0 0 0"/>
+      <geometry>
+        <sphere radius="${wheel_radius}"/>
+      </geometry>
+      <material name="green"/>
+    </visual>
+    <collision>
+      <origin xyz="0 0 0" rpy="0 0 0"/>
+      <geometry>
+        <sphere radius="${wheel_radius}"/>
+      </geometry>
+    </collision>
+  </link>
+  <joint name="chassis_caster_ball" type="continuous">
+    <parent link="chassis"/>
+    <child link="caster"/>
+    <origin xyz="${-1*rear_wheel_xoff} 0.0 ${-1*wheel_zoff}" rpy="0 0 0"/>
+  </joint>
   <xacro:wheel prefix="drivewhl_l" x_reflect="1" y_reflect="1" wheel_xoff="${drive_wheel_xoff}" joint_type="continuous"/>
   <xacro:wheel prefix="drivewhl_r" x_reflect="1" y_reflect="-1" wheel_xoff="${drive_wheel_xoff}" joint_type="continuous"/>
-  <xacro:rear_caster prefix="rearwhl_l" x_reflect="-1" y_reflect="1" wheel_xoff="${rear_wheel_xoff}" joint_type="continuous"/>
-  <xacro:rear_caster prefix="rearwhl_r" x_reflect="-1" y_reflect="-1" wheel_xoff="${rear_wheel_xoff}" joint_type="continuous"/>
+  <!--<xacro:wheel prefix="rearwhl_l" x_reflect="-1" y_reflect="1" wheel_xoff="${rear_wheel_xoff}" joint_type="continuous"/>
+  <xacro:wheel prefix="rearwhl_r" x_reflect="-1" y_reflect="-1" wheel_xoff="${rear_wheel_xoff}" joint_type="continuous"/>
+  -->
   <gazebo>
     <plugin filename="gz-sim-diff-drive-system" name="gz::sim::systems::DiffDrive">
@@ -248,6 +212,4 @@
         <topic>joint_states</topic> <joint_name>drivewhl_l_joint</joint_name>
         <joint_name>drivewhl_r_joint</joint_name>
-        <joint_name>rearwhl_l_joint</joint_name>
-        <joint_name>rearwhl_r_joint</joint_name>
     </plugin>
   </gazebo>

File: src/diy_robot_description/urdf/urdf_4wheel.urdf.xacro (robot description, xacro)
@@ -31,6 +31,5 @@
   <xacro:property name="drive_wheel_xoff" value="0.1254125"/><!-- 4.9375 inches-->
   <xacro:property name="rear_wheel_xoff" value="0.1476375"/><!-- 5.8125 inches-->
-  <xacro:property name="castor_wheel_radius" value="0.1016"/> <!-- 4-inch radius / 8-inch diameter -->
-  <xacro:property name="castor_wheel_width" value="0.0574"/> <!-- 2.26-inch STL depth -->
+  <xacro:property name="castor_wheel_radius" value="0.01"/> <!-- 3.71875 inches-->
   <xacro:property name="camera_screw_zoff" value="-0.0385"/>
   <xacro:property name="camera_screw_xoff" value="-0.007"/>
@@ -124,58 +123,4 @@
     </joint>
   </xacro:macro>
-  <!-- Rear omni wheel xacro: fixed axle, passive wheel rotation.
-       The wheel does NOT swivel. Omni behavior is approximated with
-       high friction in the rolling direction (X) and low friction
-       laterally along the axle direction (Y). -->
-  <xacro:macro name="rear_caster" params="prefix x_reflect y_reflect wheel_xoff joint_type">
-    <link name="${prefix}_link">
-      <visual>
-        <origin xyz="-0.093339143 0.185046036 -0.156049187"
-                rpy="${pi/2} 0 0"/>
-        <geometry>
-          <mesh filename="package://diy_robot_description/urdf/meshes/caster_wheel.stl"
-                scale="0.0254 0.0254 0.0254"/>
-        </geometry>
-        <material name="green"/>
-      </visual>
-      <inertial>
-        <origin xyz="0 0 0" rpy="0 0 0"/>
-        <mass value="0.6"/>
-        <inertia ixx="0.0012" ixy="0" ixz="0"
-                 iyy="0.0010" iyz="0" izz="0.0012"/>
-      </inertial>
-      <!-- Simple cylindrical collision for the omni wheel.
-           The roller effect is represented by anisotropic friction below. -->
-      <collision>
-        <origin xyz="0 0 0" rpy="${pi/2} 0 0"/>
-        <geometry>
-          <cylinder radius="${castor_wheel_radius}" length="${castor_wheel_width}"/>
-        </geometry>
-      </collision>
-    </link>
-    <!-- Fixed wheel orientation: only the wheel spins about its axle (Y). -->
-    <joint name="${prefix}_joint" type="${joint_type}">
-      <parent link="chassis"/>
-      <child link="${prefix}_link"/>
-      <origin xyz="${x_reflect*wheel_xoff} ${y_reflect*(base_width/2+wheel_ygap)} ${-wheel_zoff}" rpy="0 0 0"/>
-      <axis xyz="0 1 0"/>
-      <dynamics damping="0.02" friction="0.0"/>
-      <limit effort="20.0" velocity="20.0"/>
-    </joint>
-    <!-- Omni-wheel approximation:
-         fdir1 = chassis/wheel X direction
-         mu1   = normal rolling-direction traction
-         mu2   = very low lateral resistance along Y, emulating free rollers -->
-    <gazebo reference="${prefix}_link">
-      <material>Gazebo/Green</material>
-      <mu1>1.0</mu1>
-      <mu2>0.02</mu2>
-      <fdir1>1 0 0</fdir1>
-      <kp>1e6</kp>
-      <kd>1.0</kd>
-      <slip1>0.0</slip1>
-      <slip2>1.0</slip2>
-    </gazebo>
-  </xacro:macro>
   <link name="base_footprint">
     <inertial>
@@ -213,6 +158,6 @@
   <xacro:wheel prefix="drivewhl_l" x_reflect="1" y_reflect="1" wheel_xoff="${drive_wheel_xoff}" joint_type="continuous"/>
   <xacro:wheel prefix="drivewhl_r" x_reflect="1" y_reflect="-1" wheel_xoff="${drive_wheel_xoff}" joint_type="continuous"/>
-  <xacro:rear_caster prefix="rearwhl_l" x_reflect="-1" y_reflect="1" wheel_xoff="${rear_wheel_xoff}" joint_type="continuous"/>
-  <xacro:rear_caster prefix="rearwhl_r" x_reflect="-1" y_reflect="-1" wheel_xoff="${rear_wheel_xoff}" joint_type="continuous"/>
+  <xacro:wheel prefix="rearwhl_l" x_reflect="-1" y_reflect="1" wheel_xoff="${rear_wheel_xoff}" joint_type="continuous"/>
+  <xacro:wheel prefix="rearwhl_r" x_reflect="-1" y_reflect="-1" wheel_xoff="${rear_wheel_xoff}" joint_type="continuous"/>
   <gazebo>
     <plugin filename="gz-sim-diff-drive-system" name="gz::sim::systems::DiffDrive">
