Commit message: Added imu and lidar to the simulator

File: src/diy_robot_description/urdf/imu.urdf.xacro (robot description, xacro)
@@ -42,8 +42,8 @@
       <sensor type="imu" name="imu_sensor">
         <always_on>1</always_on>
-        <update_rate>50</update_rate>
+        <update_rate>100</update_rate>
         <visualize>true</visualize>
         <topic>imu</topic>
-        <frame_name>imu_link</frame_name>
+        <ignition_frame_id>imu_link</ignition_frame_id>
         <plugin filename="ignition-gazebo-imu-system" name="ignition::gazebo::systems::Imu">
         </plugin>

File: src/diy_robot_description/urdf/lidar.urdf.xacro (robot description, xacro)
@@ -19,5 +19,5 @@
         <origin xyz="0 0 0" rpy="0 0 0"/>
         <geometry>
-          <mesh filename="package:/diy_robot_description/urdf/meshes/lidar_3d_v1.dae"/>
+          <mesh filename="package://diy_robot_description/urdf/meshes/lidar_3d_v1.dae"/>
         </geometry>
       </visual>
@@ -36,4 +36,5 @@
         <visualize>true</visualize>
         <topic>lidar</topic>
+        <ignition_frame_id>lidar_link</ignition_frame_id>
         <ray>
           <scan>
@@ -45,5 +46,5 @@
             </horizontal>
             <vertical>
-              <samples>16</samples>
+              <samples>32</samples>
               <resolution>1</resolution>
               <min_angle>-0.2618</min_angle>
@@ -53,5 +54,5 @@
           <range>
             <min>0.08</min>
-            <max>10.0</max>
+            <max>30.0</max>
             <resolution>0.01</resolution>
           </range>

File: src/diy_robot_description/urdf/robot.urdf.xacro (robot description, xacro)
@@ -31,4 +31,5 @@
   <xacro:property name="drive_wheel_xoff" value="0.1254125"/><!-- 4.9375 inches-->
   <xacro:property name="rear_wheel_xoff" value="0.1476375"/><!-- 5.8125 inches-->
+  <xacro:property name="castor_wheel_radius" value="0.01"/> <!-- 3.71875 inches-->
   <xacro:property name="camera_screw_zoff" value="-0.0385"/>
   <xacro:property name="camera_screw_xoff" value="-0.007"/>
@@ -53,5 +54,5 @@
   </xacro:imu_v1>
   <material name="transparent_blue">
-    <color rgba="0.0 0.0 1.0 0.25"/>
+    <color rgba="0.0 0.0 1.0 0.75"/>
   </material>
   <material name="blue">
@@ -136,5 +137,5 @@
         <box size="${base_length} ${base_width} ${base_height}"/>
       </geometry>
-      <material name="transparent_blue"/>
+      <material name="blue"/>
     </visual>
     <collision>
@@ -145,8 +146,62 @@
     </collision>
   </link>
+  <link name="caster">
+    <inertial>
+      <origin xyz="0 0 0" rpy="0 0 0"/>
+      <mass value="1.0"/>
+      <inertia ixx="0.1" ixy="0.0" ixz="0.0" iyy="0.1" iyz="0.0" izz="0.1"/>
+    </inertial>
+    <visual>
+      <origin xyz="0 0 0" rpy="0 0 0"/>
+      <geometry>
+        <sphere radius="${wheel_radius}"/>
+      </geometry>
+      <material name="green"/>
+    </visual>
+    <collision>
+      <origin xyz="0 0 0" rpy="0 0 0"/>
+      <geometry>
+        <sphere radius="${wheel_radius}"/>
+      </geometry>
+    </collision>
+  </link>
+  <joint name="chassis_caster_ball" type="continuous">
+    <parent link="chassis"/>
+    <child link="caster"/>
+    <origin xyz="${-1*rear_wheel_xoff} 0.0 ${-1*wheel_zoff}" rpy="0 0 0"/>
+  </joint>
   <xacro:wheel prefix="drivewhl_l" x_reflect="1" y_reflect="1" wheel_xoff="${drive_wheel_xoff}" joint_type="continuous"/>
   <xacro:wheel prefix="drivewhl_r" x_reflect="1" y_reflect="-1" wheel_xoff="${drive_wheel_xoff}" joint_type="continuous"/>
-  <xacro:wheel prefix="rearwhl_l" x_reflect="-1" y_reflect="1" wheel_xoff="${rear_wheel_xoff}" joint_type="continuous"/>
+  <!--<xacro:wheel prefix="rearwhl_l" x_reflect="-1" y_reflect="1" wheel_xoff="${rear_wheel_xoff}" joint_type="continuous"/>
   <xacro:wheel prefix="rearwhl_r" x_reflect="-1" y_reflect="-1" wheel_xoff="${rear_wheel_xoff}" joint_type="continuous"/>
+  -->
+  <gazebo>
+    <plugin filename="gz-sim-diff-drive-system" name="gz::sim::systems::DiffDrive">
+        <left_joint>drivewhl_l_joint</left_joint>
+        <right_joint>drivewhl_r_joint</right_joint>
+        <wheel_separation>${base_width+2*wheel_ygap}</wheel_separation> <!-- Adjust to your robot's width (meters) -->
+        <wheel_radius>${wheel_radius}</wheel_radius>     <!-- Adjust to your wheel radius (meters) -->
+        <topic>cmd_vel</topic>
+        <robot_param_node>/robot_state_publisher</robot_param_node>
+    </plugin>
+  </gazebo>
+  <gazebo>
+    <plugin filename="gz-sim-joint-state-publisher-system" name="gz::sim::systems::JointStatePublisher">
+        <topic>joint_states</topic> <joint_name>drivewhl_l_joint</joint_name>
+        <joint_name>drivewhl_r_joint</joint_name>
+    </plugin>
+  </gazebo>
+   <!-- INSERT GROUND TRUTH POSE PUBLISHER HERE -->
+  <gazebo>
+    <plugin filename="libignition-gazebo-pose-publisher-system.so"
+          name="ignition::gazebo::systems::PosePublisher">
+      <publish_link_pose>false</publish_link_pose>
+      <publish_visual_pose>false</publish_visual_pose>
+      <publish_nested_model_pose>true</publish_nested_model_pose>
+      <use_pose_vector_msg>true</use_pose_vector_msg>
+      <static_publisher>false</static_publisher>
+      <publish_model_pose>true</publish_model_pose>
+    </plugin>
+  </gazebo>
 <!--
   <link name="wheel_1">

Commit message: Include the gazebo plugins in the xacro only when the sim flag is true. If the sim flag is false, plugins are not needed

File: src/diy_robot_description/urdf/imu.urdf.xacro (robot description, xacro)
@@ -39,15 +39,17 @@
     </gazebo>
     -->
-    <gazebo reference="imu_link">
-      <sensor type="imu" name="imu_sensor">
-        <always_on>1</always_on>
-        <update_rate>100</update_rate>
-        <visualize>true</visualize>
-        <topic>imu</topic>
-        <ignition_frame_id>imu_link</ignition_frame_id>
-        <plugin filename="ignition-gazebo-imu-system" name="ignition::gazebo::systems::Imu">
-        </plugin>
-      </sensor>
-    </gazebo>
+    <xacro:if value="$(arg sim)">
+      <gazebo reference="imu_link">
+        <sensor type="imu" name="imu_sensor">
+          <always_on>1</always_on>
+          <update_rate>100</update_rate>
+          <visualize>true</visualize>
+          <topic>imu</topic>
+          <ignition_frame_id>imu_link</ignition_frame_id>
+          <plugin filename="ignition-gazebo-imu-system" name="ignition::gazebo::systems::Imu">
+          </plugin>
+        </sensor>
+      </gazebo>
+    </xacro:if>
   </xacro:macro>
 </robot>

File: src/diy_robot_description/urdf/lidar.urdf.xacro (robot description, xacro)
@@ -29,4 +29,5 @@
       </collision>
     </link>
+    <xacro:if value="$(arg sim)">
     <gazebo reference="lidar_link">
       <sensor type="gpu_lidar" name="gpu_lidar">
@@ -69,4 +70,5 @@
       </sensor>
     </gazebo>
+    </xacro:if>
   </xacro:macro>
 </robot>

File: src/diy_robot_description/urdf/original.urdf.xacro (robot description, xacro)
@@ -44,4 +44,5 @@
   <xacro:property name="hesai_centroid_z" value="0.0124"/>
   <xacro:arg name="use_nominal_extrinsics" default="true" />
+  <xacro:arg name="sim" default="false" />
   <xacro:include filename="lidar.urdf.xacro" />
   <xacro:include filename="imu.urdf.xacro" />

File: src/diy_robot_description/urdf/robot.urdf.xacro (robot description, xacro)
@@ -28,5 +28,5 @@
   <xacro:property name="base_height" value="0.174625"/> <!-- 6.875 inches-->
   <xacro:property name="pool_noodle_radius" value="0.047625"/> <!-- 1.875 inches-->
-  <xacro:property name="castor_wheel_width" value="0.0574"/> <!-- 2.26-inch STL depth -->
+  <xacro:property name="castor_wheel_width" value="0.04305"/> <!-- 2.26-inch STL depth; old value 0.0574 -->
   <xacro:property name="wheel_radius" value="0.0762"/> <!-- 3 inches-->
   <xacro:property name="wheel_width" value="0.0254"/><!-- 1 inches-->
@@ -52,4 +52,6 @@
   <xacro:property name="hesai_centroid_z" value="0.0124"/>
   <xacro:arg name="use_nominal_extrinsics" default="true" />
+  <!-- sim:=true (pass via `xacro robot.urdf.xacro sim:=true`) includes all Gazebo plugins/tags -->
+  <xacro:arg name="sim" default="false" />
   <xacro:include filename="lidar.urdf.xacro" />
   <xacro:include filename="imu.urdf.xacro" />
@@ -116,15 +118,17 @@
       </collision>
     </link>
-    <gazebo reference="${prefix}_link">
-        <material>Gazebo/Red</material>
-        <mu1>1.5</mu1>
-        <mu2>1.5</mu2>
-        <kp>1e6</kp>
-        <kd>1.0</kd>
-    </gazebo>
+    <xacro:if value="$(arg sim)">
+      <gazebo reference="${prefix}_link">
+          <material>Gazebo/Red</material>
+          <mu1>1.5</mu1>
+          <mu2>1.5</mu2>
+          <kp>1e6</kp>
+          <kd>1.0</kd>
+      </gazebo>
+    </xacro:if>
     <joint name="${prefix}_joint" type="${joint_type}">
       <parent link="base_link"/>
       <child link="${prefix}_link"/>
-      <origin xyz="${x_reflect*wheel_xoff} ${y_reflect*(base_width/2+wheel_ygap)} ${-wheel_zoff}" rpy="0 0 0"/>
+      <origin xyz="${x_reflect*wheel_xoff} ${y_reflect*(base_width/2+wheel_ygap)} 0.0" rpy="0 0 0"/>
       <axis xyz="0 1 0"/>
       <limit effort="20.0" velocity="10.0"/>
@@ -138,9 +142,9 @@
     <link name="${prefix}_link">
       <visual>
-        <origin xyz="-0.093339143 0.185046036 -0.156049187"
-                rpy="${pi/2} 0 0"/>
+        <!-- <origin xyz="-0.093339143 0.185046036 -0.156049187" rpy="${pi/2} 0 0"/> -->
+        <origin xyz="-0.07000435725  0.138784527 -0.11703689025" rpy="${pi/2} 0 0"/>
         <geometry>
           <mesh filename="package://diy_robot_description/urdf/meshes/caster_wheel.stl"
-                scale="0.0254 0.0254 0.0254"/>
+                scale="0.01905 0.01905 0.01905"/>
         </geometry>
         <material name="green"/>
@@ -163,7 +167,7 @@
     <!-- Fixed wheel orientation: only the wheel spins about its axle (Y). -->
     <joint name="${prefix}_joint" type="${joint_type}">
-      <parent link="chassis"/>
+      <parent link="base_link"/>
       <child link="${prefix}_link"/>
-      <origin xyz="${x_reflect*wheel_xoff} ${y_reflect*(base_width/2+wheel_ygap)} ${-wheel_zoff}" rpy="0 0 0"/>
+      <origin xyz="${x_reflect*wheel_xoff} ${y_reflect*(base_width/2+wheel_ygap)} 0.0" rpy="0 0 0"/>
       <axis xyz="0 1 0"/>
       <dynamics damping="0.02" friction="0.0"/>
@@ -174,23 +178,18 @@
          mu1   = normal rolling-direction traction
          mu2   = very low lateral resistance along Y, emulating free rollers -->
-    <gazebo reference="${prefix}_link">
-      <material>Gazebo/Green</material>
-      <mu1>1.0</mu1>
-      <mu2>0.02</mu2>
-      <fdir1>1 0 0</fdir1>
-      <kp>1e6</kp>
-      <kd>1.0</kd>
-      <slip1>0.0</slip1>
-      <slip2>1.0</slip2>
-    </gazebo>
+    <xacro:if value="$(arg sim)">
+      <gazebo reference="${prefix}_link">
+        <material>Gazebo/Green</material>
+        <mu1>1.0</mu1>
+        <mu2>0.02</mu2>
+        <fdir1>1 0 0</fdir1>
+        <kp>1e6</kp>
+        <kd>1.0</kd>
+        <slip1>0.0</slip1>
+        <slip2>1.0</slip2>
+      </gazebo>
+    </xacro:if>
   </xacro:macro>
-  <link name="base_footprint">
-    <inertial>
-      <mass value="0.001"/>
-      <inertia ixx="1e-06" ixy="0.0" ixz="0.0"
-               iyy="1e-06" iyz="0.0"
-               izz="1e-06"/>
-    </inertial>
-  </link>
+  <link name="base_footprint"/>
   <joint name="base_footprint_to_base_link" type="fixed">
     <parent link="base_footprint"/>
@@ -198,5 +197,27 @@
     <origin xyz="0 0 ${wheel_radius}" rpy="0 0 0"/>
   </joint>
-  <link name="base_link"/>
+  <link name="base_link">
+      <inertial>
+      <origin xyz="${AR_from_front-base_length/2} 0 ${base_height/2+base_off_ground-wheel_radius}" rpy="0 0 0"/> <!-- change based on TF -->
+      <mass value="${body_mass}"/>
+      <inertia ixx="${body_mass * (base_width**2 + base_height**2)/12.0 + body_mass * (base_height/2+base_off_ground-wheel_radius)**2}" ixy="0.0" ixz="0.0"
+               iyy="${body_mass * (base_length**2 + base_height**2)/12.0 + body_mass * ((AR_from_front-base_length/2)**2 + (base_height/2+base_off_ground-wheel_radius)**2)}" iyz="0.0"
+               izz="${body_mass * (base_length**2 + base_width**2)/12.0 + body_mass * (AR_from_front-base_length/2)**2}"/>
+    </inertial>
+    <visual>
+      <origin xyz="${AR_from_front-base_length/2} 0 ${base_height/2+base_off_ground-wheel_radius}" rpy="0 0 0"/>
+      <geometry>
+        <box size="${base_length} ${base_width} ${base_height}"/>
+      </geometry>
+      <material name="blue"/>
+    </visual>
+    <collision>
+      <origin xyz="${AR_from_front-base_length/2} 0 ${base_height/2+base_off_ground-wheel_radius}" rpy="0 0 0"/> <!-- change based on TF -->
+      <geometry>
+        <box size="${base_length} ${base_width} ${base_height}"/>
+      </geometry>
+    </collision>
+  </link>
+<!--
   <joint name="base_link_to_chassis" type="fixed">
     <parent link="base_link"/>
@@ -206,5 +227,5 @@
   <link name="chassis">
     <inertial>
-      <origin xyz="${AR_from_front-base_length/2} 0 ${base_height/2+base_off_ground-wheel_radius}" rpy="0 0 0"/> <!-- change based on TF -->
+      <origin xyz="${AR_from_front-base_length/2} 0 ${base_height/2+base_off_ground-wheel_radius}" rpy="0 0 0"/>
       <mass value="${body_mass}"/>
       <inertia ixx="0.5 * body_mass * (base_width * base_width + base_height * base_height)" ixy="0.0" ixz="0.0"
@@ -220,5 +241,5 @@
     </visual>
     <collision>
-      <origin xyz="${AR_from_front-base_length/2} 0 ${base_height/2+base_off_ground-wheel_radius}" rpy="0 0 0"/> <!-- change based on TF -->
+      <origin xyz="${AR_from_front-base_length/2} 0 ${base_height/2+base_off_ground-wheel_radius}" rpy="0 0 0"/>
       <geometry>
         <box size="${base_length} ${base_width} ${base_height}"/>
@@ -226,57 +247,61 @@
     </collision>
   </link>
+-->
   <xacro:wheel prefix="drivewhl_l" x_reflect="1" y_reflect="1" wheel_xoff="${drive_wheel_xoff}" joint_type="continuous"/>
   <xacro:wheel prefix="drivewhl_r" x_reflect="1" y_reflect="-1" wheel_xoff="${drive_wheel_xoff}" joint_type="continuous"/>
   <xacro:rear_caster prefix="rearwhl_l" x_reflect="-1" y_reflect="1" wheel_xoff="${rear_wheel_xoff}" joint_type="continuous"/>
   <xacro:rear_caster prefix="rearwhl_r" x_reflect="-1" y_reflect="-1" wheel_xoff="${rear_wheel_xoff}" joint_type="continuous"/>
-  <gazebo>
-    <plugin filename="gz-sim-diff-drive-system" name="gz::sim::systems::DiffDrive">
-        <left_joint>drivewhl_l_joint</left_joint>
-        <right_joint>drivewhl_r_joint</right_joint>
-        <wheel_separation>${base_width+2*wheel_ygap}</wheel_separation> <!-- Adjust to your robot's width (meters) -->
-        <wheel_radius>${wheel_radius}</wheel_radius>     <!-- Adjust to your wheel radius (meters) -->
-        <topic>cmd_vel</topic>
-        <odom_topic>odom_wheel</odom_topic>   <!-- wheel encoder odom — drifts on ramp/slip -->
-        <!-- Publish odom→base_footprint TF — must match Nav2 robot_base_frame.
-             Ignition namespaces these as diy_robot/odom→diy_robot/base_footprint.
-             SIM only: on real robot EKF1/EKF2 publish this transform instead. -->
-        <odom_frame>odom</odom_frame>
-        <robot_base_frame>base_footprint</robot_base_frame>
-        <tf_topic>/tf</tf_topic>
-        <robot_param_node>/robot_state_publisher</robot_param_node>
-    </plugin>
-  </gazebo>
-  <!-- SIM ONLY: Ground-truth odometry from Gazebo physics engine.
-       Publishes perfect pose to /odom — no wheel slip drift.
-       On real robot: EKF2 fuses wheel + IMU + NDT into /odometry/filtered instead. -->
-  <gazebo>
-    <plugin filename="gz-sim-odometry-publisher-system" name="gz::sim::systems::OdometryPublisher">
-        <odom_frame>odom</odom_frame>
-        <robot_base_frame>base_footprint</robot_base_frame>
-        <odom_topic>/odom</odom_topic>
-        <tf_topic>/tf</tf_topic>
-        <odom_publish_frequency>50</odom_publish_frequency>
-    </plugin>
-  </gazebo>
-  <gazebo>
-    <plugin filename="gz-sim-joint-state-publisher-system" name="gz::sim::systems::JointStatePublisher">
-        <topic>joint_states</topic> <joint_name>drivewhl_l_joint</joint_name>
-        <joint_name>drivewhl_r_joint</joint_name>
-        <joint_name>rearwhl_l_joint</joint_name>
-        <joint_name>rearwhl_r_joint</joint_name>
-    </plugin>
-  </gazebo>
-   <!-- INSERT GROUND TRUTH POSE PUBLISHER HERE -->
-  <gazebo>
-    <plugin filename="libignition-gazebo-pose-publisher-system.so"
-          name="ignition::gazebo::systems::PosePublisher">
-      <publish_link_pose>false</publish_link_pose>
-      <publish_visual_pose>false</publish_visual_pose>
-      <publish_nested_model_pose>true</publish_nested_model_pose>
-      <use_pose_vector_msg>true</use_pose_vector_msg>
-      <static_publisher>false</static_publisher>
-      <publish_model_pose>true</publish_model_pose>
-    </plugin>
-  </gazebo>
+  <xacro:if value="$(arg sim)">
+    <gazebo>
+      <plugin filename="gz-sim-diff-drive-system" name="gz::sim::systems::DiffDrive">
+          <left_joint>drivewhl_l_joint</left_joint>
+          <right_joint>drivewhl_r_joint</right_joint>
+          <wheel_separation>${base_width+2*wheel_ygap}</wheel_separation> <!-- Adjust to your robot's width (meters) -->
+          <wheel_radius>${wheel_radius}</wheel_radius>     <!-- Adjust to your wheel radius (meters) -->
+          <topic>cmd_vel</topic>
+          <odom_topic>odom_wheel</odom_topic>   <!-- wheel encoder odom — drifts on ramp/slip -->
+          <!-- Publish odom→base_footprint TF — must match Nav2 robot_base_frame.
+               Ignition namespaces these as diy_robot/odom→diy_robot/base_footprint.
+               SIM only: on real robot EKF1/EKF2 publish this transform instead. -->
+          <odom_frame>odom</odom_frame>
+          <robot_base_frame>base_footprint</robot_base_frame>
+          <tf_topic>/tf</tf_topic>
+          <robot_param_node>/robot_state_publisher</robot_param_node>
+      </plugin>
+    </gazebo>
+    <!-- SIM ONLY: Ground-truth odometry from Gazebo physics engine.
+         Publishes perfect pose to /odom — no wheel slip drift.
+         On real robot: EKF2 fuses wheel + IMU + NDT into /odometry/filtered instead. -->
+    <gazebo>
+      <plugin filename="gz-sim-odometry-publisher-system" name="gz::sim::systems::OdometryPublisher">
+          <odom_frame>odom</odom_frame>
+          <robot_base_frame>base_footprint</robot_base_frame>
+          <odom_topic>/odom</odom_topic>
+          <tf_topic>/tf</tf_topic>
+          <odom_publish_frequency>50</odom_publish_frequency>
+      </plugin>
+    </gazebo>
+    <gazebo>
+      <plugin filename="gz-sim-joint-state-publisher-system" name="gz::sim::systems::JointStatePublisher">
+          <topic>joint_states</topic>
+          <joint_name>drivewhl_l_joint</joint_name>
+          <joint_name>drivewhl_r_joint</joint_name>
+          <joint_name>rearwhl_l_joint</joint_name>
+          <joint_name>rearwhl_r_joint</joint_name>
+      </plugin>
+    </gazebo>
+     <!-- INSERT GROUND TRUTH POSE PUBLISHER HERE -->
+    <gazebo>
+      <plugin filename="libignition-gazebo-pose-publisher-system.so"
+            name="ignition::gazebo::systems::PosePublisher">
+        <publish_link_pose>false</publish_link_pose>
+        <publish_visual_pose>false</publish_visual_pose>
+        <publish_nested_model_pose>true</publish_nested_model_pose>
+        <use_pose_vector_msg>true</use_pose_vector_msg>
+        <static_publisher>false</static_publisher>
+        <publish_model_pose>true</publish_model_pose>
+      </plugin>
+    </gazebo>
+  </xacro:if>
 <!--
   <link name="wheel_1">

File: src/diy_robot_description/urdf/urdf_4wheel.urdf.xacro (robot description, xacro)
@@ -44,4 +44,5 @@
   <xacro:property name="hesai_centroid_z" value="0.0124"/>
   <xacro:arg name="use_nominal_extrinsics" default="true" />
+  <xacro:arg name="sim" default="false" />
   <xacro:include filename="lidar.urdf.xacro" />
   <xacro:include filename="imu.urdf.xacro" />
