Commit message: rename folders

File: src/robot_description/urdf/lidar.urdf.xacro (robot description, xacro)
@@ -19,5 +19,5 @@
         <origin xyz="0 0 0" rpy="0 0 0"/>
         <geometry>
-          <mesh filename="package://diy_robot_description/urdf/meshes/lidar_3d_v1.dae"/>
+          <mesh filename="package://robot_description/urdf/meshes/lidar_3d_v1.dae"/>
         </geometry>
       </visual>

File: src/robot_description/urdf/robot.urdf.xacro (robot description, xacro)
@@ -151,5 +151,5 @@
         <origin xyz="-0.07000435725  0.138784527 -0.11703689025" rpy="${pi/2} 0 0"/>
         <geometry>
-          <mesh filename="package://diy_robot_description/urdf/meshes/caster_wheel.stl"
+          <mesh filename="package://robot_description/urdf/meshes/caster_wheel.stl"
                 scale="0.01905 0.01905 0.01905"/>
         </geometry>
@@ -270,5 +270,5 @@
           <odom_topic>odom_wheel</odom_topic>   <!-- wheel encoder odom — drifts on ramp/slip -->
           <!-- Publish odom→base_link TF — must match Nav2 robot_base_frame.
-               Ignition namespaces these as diy_robot/odom→diy_robot/base_link.
+               Ignition namespaces these as robot/odom→robot/base_link.
                SIM only: on real robot EKF1/EKF2 publish this transform instead. -->
           <odom_frame>odom</odom_frame>

Commit message: Fast Lio Working, Loop PGO WIP

File: src/robot_description/urdf/lidar.urdf.xacro (robot description, xacro)
@@ -5,7 +5,7 @@
       <xacro:insert_block name="origin" />
       <parent link="${parent}"/>
-      <child link="lidar_link"/>
+      <child link="hesai_lidar"/>
     </joint>
-    <link name="lidar_link">
+    <link name="hesai_lidar">
       <inertial>
         <origin xyz="0 0 0" rpy="0 0 0"/>
@@ -30,5 +30,5 @@
     </link>
     <xacro:if value="$(arg sim)">
-    <gazebo reference="lidar_link">
+    <gazebo reference="hesai_lidar">
       <sensor type="gpu_lidar" name="gpu_lidar">
         <pose>0 0 0 0 0 0</pose>
@@ -37,5 +37,5 @@
         <visualize>false</visualize>
         <topic>lidar</topic>
-        <ignition_frame_id>lidar_link</ignition_frame_id>
+        <ignition_frame_id>hesai_lidar</ignition_frame_id>
         <ray>
           <scan>
@@ -65,5 +65,5 @@
           </ros>
           <output_type>sensor_msgs/PointCloud2</output_type>
-          <frame_name>lidar_link</frame_name>
+          <frame_name>hesai_lidar</frame_name>
         </plugin>
         -->

File: src/robot_description/urdf/robot.urdf.xacro (robot description, xacro)
@@ -11,5 +11,5 @@
           └── base_footprint  (published by the single EKF via /odometry/filtered)
                └──base_link  (published by URDF via robot_state_publisher)
-                    ├── lidar_link   <- REAL, measured offset (see lidar.urdf.xacro)
+                    ├── hesai_lidar   <- REAL, measured offset (see lidar.urdf.xacro)
                     ├── imu_link     <- REAL, measured offset (see imu.urdf.xacro)
                     ├── camera_link  <- NOT YET DEFINED in this file — see
