Commit message: Updated urdf xacro

File: src/robot_description/urdf/ackermann_robot.urdf.xacro (robot description, xacro)
@@ -8,12 +8,12 @@
   <xacro:property name="W" value="0.055" /> <!-- 55 mm Wheel Width -->
   <xacro:property name="R" value="0.0675" /> <!-- 67.5 mm Wheel Radius -->
-  <xacro:property name="X_OFFSET" value="0.2" /> <!-- 67.5 mm Wheel Radius -->
-  <xacro:property name="H" value="0.1" /> <!-- 67.5 mm Wheel Radius -->
+  <xacro:property name="X_OFFSET" value="0.2" />
+  <xacro:property name="H" value="0.1905" /> <!-- 7.5 inches Wheel Radius -->
   <xacro:property name="chassis_mass" value="10.0" />
   <xacro:property name="wheel_mass" value="1.0" />
   <xacro:property name="total_mass" value="1.0" />
-  <xacro:property name="Lower_angle_limit" value="-0.6" />
-  <xacro:property name="Upper_angle_limit" value="0.6" />
-  <xacro:property name="velocity" value="1.0" />
+  <xacro:property name="Lower_angle_limit" value="-0.5" />
+  <xacro:property name="Upper_angle_limit" value="0.5" />
+  <xacro:property name="velocity" value="3.0" />
   <xacro:property name="Effort" value="10.0" />
   <xacro:property name="Wheel_y_inertia" value="${wheel_mass * R * R/2.0}" />
@@ -202,5 +202,5 @@
     <parent link="base_link"/>
     <child link="hesai_lidar"/>
-    <origin xyz="${B/2} 0 ${H + 0.05}" rpy="0 0 0"/>
+    <origin xyz="${B} 0 ${H + 0.05}" rpy="0 0 0"/>
   </joint>
   <link name="hesai_lidar">
@@ -218,7 +218,8 @@
     <parent link="base_link"/>
     <child link="imu_link"/>
-    <origin xyz="${B/2} 0 ${H/2}" rpy="0 0 0"/>
+    <origin xyz="${B} 0 0.1016" rpy="0 0 0"/> <!--${B} 0 ${H/2} --> <!-- 0.1016 is the height of imu from the center of the wheel
   </joint>
   <link name="imu_link"/>
+<!--
   <ros2_control name="AckermannRobotHardware" type="system">
     <hardware>
@@ -239,5 +240,4 @@
       <param name="supply_current_limit">20.0</param>
     </hardware>
-  <!-- Traction Wheels (Rear) -->
   <joint name="rear_left_wheel_joint">
     <command_interface name="velocity"/>
@@ -250,5 +250,4 @@
     <state_interface name="position"/>
   </joint>
-  <!-- Steering Knuckles (Front) -->
   <joint name="front_left_steer_joint">
     <command_interface name="position"/>
@@ -260,3 +259,4 @@
   </joint>
 </ros2_control>
+-->
 </robot>

Commit message: latest changes - zed2i implemt on fastLio, plan-B addition, waypoint-seq update

File: src/robot_description/urdf/ackermann_robot.urdf.xacro (robot description, xacro)
@@ -214,11 +214,18 @@
     </visual>
   </link>
+  <link name="imu_link"/>
   <!-- IMU Link (Adjust location relative to base_link center) -->
   <joint name="imu_joint" type="fixed">
     <parent link="base_link"/>
     <child link="imu_link"/>
-    <origin xyz="${B} 0 0.1016" rpy="0 0 0"/> <!--${B} 0 ${H/2} --> <!-- 0.1016 is the height of imu from the center of the wheel
-  </joint>
-  <link name="imu_link"/>
+    <origin xyz="${B} 0 0.1016" rpy="0 0 0"/> <!--${B} 0 ${H/2} --> <!-- 0.1016 is the height of imu from the center of the wheel -->
+  </joint>
+  <link name="zed_camera_link"/>
+  <joint name="base_to_camera_joint" type="fixed">
+    <parent link="base_link"/>
+    <child link="zed_camera_link"/>
+    <origin xyz="${B + 0.05} 0.0 0.1484" rpy="0 0 0"/>
+  </joint>
+</robot>
 <!--
   <ros2_control name="AckermannRobotHardware" type="system">
@@ -260,3 +267,2 @@
 </ros2_control>
 -->
-</robot>

Commit message: latest changes to mcd-3dl and lio localization

File: src/robot_description/urdf/ackermann_robot.urdf.xacro (robot description, xacro)
@@ -225,5 +225,5 @@
     <parent link="base_link"/>
     <child link="zed_camera_link"/>
-    <origin xyz="${B + 0.05} 0.0 0.1484" rpy="0 0 0"/>
+    <origin xyz="${B + 0.05} 1.0 0.1484" rpy="0 0 0"/>
   </joint>
 </robot>

Commit message: added single launch for obstacle, mcl_3dl fixes, relay node fixes, launch fixes

File: src/robot_description/urdf/ackermann_robot.urdf.xacro (robot description, xacro)
@@ -225,5 +225,5 @@
     <parent link="base_link"/>
     <child link="zed_camera_link"/>
-    <origin xyz="${B + 0.05} 1.0 0.1484" rpy="0 0 0"/>
+    <origin xyz="${B + 0.05} 0.0 0.1484" rpy="0 0 0"/>
   </joint>
 </robot>
